File: hardware/keyboard.kicad_sch (KiCad schematic)
At the start: 82 parts, among them J1 BATT, J2 nice!view, SW1 PLAY/PAUSE, SW10 NEXT, SW11 TAB, SW12 Q, SW13 W, SW14 E, SW15 R, SW16 T, SW17 CAPS, SW18 A, SW19 S, SW2 TILDA, SW20 D, SW21 F, SW22 G, SW23 M2, SW24 SHIFT, SW25 Z, SW26 X, SW27 C, SW28 V, SW29 B, SW3 1, SW30 ALT_1, SW31 FN, SW32 CONTROL, SW33 OPTION, SW34 COMMAND, SW35 SPACE, SW4 2, SW5 3, SW6 4, SW7 5, SW8 ON_OFF, SW9 NRST, U1 nice!nano

Commit message: finish right keyboard, generate 3D models, add distribution folders
Parts:
- J1: footprint Connector_JST:JST_ZH_B2B-ZR_1x02_P1.50mm_Vertical -> Connector_JST:JST_PH_S2B-PH-K_1x02_P2.00mm_Horizontal
- SW8: footprint Button_Switch_THT:SW_Slide_SPDT_Angled_CK_OS102011MA1Q -> ScottoKeebs_Components:Switch_MSK12C02
Changed lines of the file:
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@@
 			)
 		)
-		(property "Footprint" "Button_Switch_THT:SW_Slide_SPDT_Angled_CK_OS102011MA1Q"
+		(property "Footprint" "ScottoKeebs_Components:Switch_MSK12C02"
 			(at 220.98 42.672 0)
 			(effects
@@
 			)
 		)
-		(property "Footprint" "Connector_JST:JST_ZH_B2B-ZR_1x02_P1.50mm_Vertical"
+		(property "Footprint" "Connector_JST:JST_PH_S2B-PH-K_1x02_P2.00mm_Horizontal"
 			(at 236.22 31.75 0)
 			(effects
