File: hardware/keyboard-right.kicad_pcb (KiCad board)
At the start: 2 copper layers, 140.3 x 111.5 mm, 83 parts, among them J1 BATT, J2 nice!view, SW1 ON/OFF, SW10 U, SW11 I, SW12 O, SW13 P, SW14 {, SW15 H, SW16 J, SW17 K, SW18 L, SW19 ;, SW2 NRST, SW20 ', SW21 __ENTER, SW22 N, SW23 M, SW24 ,, SW25 ., SW26 /, SW27 SHIFT, SW28 UP, SW29 M1, SW3 6, SW30 DOWN, SW31 LEFT, SW32 ALT_2, SW33 RIGHT, SW34 DEL, SW35 }, SW36 SPACE, SW4 7, SW5 8, SW6 9, SW7 0, SW8 -, SW9 Y, U1 nice!nano

Commit message: finish right keyboard, generate 3D models, add distribution folders
Parts:
- added G***: LOGO, Synth:lenimal_logo_full, F.Cu at (52.2, 101.5)
- added G***: LOGO, Synth:lenimal_logo_full, B.Cu at (52.2, 101.5)
- added H11: MountingHole, keyboard:MountingPin_M2, F.Cu at (55.2, 160.0)
- added H12: MountingHole, keyboard:MountingPin_M2, F.Cu at (200.5, 143.0)
- added H13: MountingHole, keyboard:MountingPin_M3, F.Cu at (61.8, 90.2)
- added H14: MountingHole, keyboard:MountingPin_M2, F.Cu at (200.5, 58.0)
- added H15: MountingHole, keyboard:MountingPin_M2, F.Cu at (36.8, 128.5)
- added J4: NUM_PAD_ROWS, Connector_PinHeader_2.54mm:PinHeader_1x05_P2.54mm_Horizontal, F.Cu at (201.0, 128.0)
- added J5: NUM_PAD_COLUMNS, Connector_PinHeader_2.54mm:PinHeader_1x05_P2.54mm_Horizontal, F.Cu at (201.0, 62.0)
- H1, H10, H3, H4: footprint MountingHole:MountingHole_3.2mm_M3 -> keyboard:MountingPin_M3
- H2, H5, H6, H7, H8, H9: footprint MountingHole:MountingHole_2.2mm_M2 -> keyboard:MountingPin_M2
- J1: footprint Connector_JST:JST_ZH_B2B-ZR_1x02_P1.50mm_Vertical -> Connector_JST:JST_PH_S2B-PH-K_1x02_P2.00mm_Horizontal; moved to B.Cu
- SW1: value ON/OFF -> SW_SPDT; footprint Button_Switch_THT:SW_Slide_SPDT_Angled_CK_OS102011MA1Q -> ScottoKeebs_Components:Switch_MSK12C02
- moved D30 302.3 mm to (59.3, 131.2), turned to 120 degrees
- moved D34 294.4 mm to (67.7, 145.9), turned to 120 degrees
- moved D27 290.6 mm to (71.0, 119.1), turned to 90 degrees
- moved SW2 277.9 mm to (75.0, 55.0)
- moved H10 276.5 mm to (70.2, 126.2)
- moved SW32 273.5 mm to (49.8, 133.0), turned to 30 degrees
- moved J2 272.8 mm to (54.0, 86.0), turned to 90 degrees
- moved D13 260.6 mm to (89.0, 104.9), turned to 90 degrees
- moved H4 260.5 mm to (90.0, 142.5)
- moved D20 258.6 mm to (89.0, 122.0), turned to 90 degrees
- moved SW1 256.0 mm to (84.8, 51.6)
- moved SW36 254.8 mm to (58.3, 147.8), turned to 30 degrees
- moved J1 250.2 mm to (91.8, 52.8), turned to -90 degrees
- moved H8 248.6 mm to (89.0, 94.2)
- moved D1 242.1 mm to (89.0, 70.8), turned to 90 degrees
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Connections:
- SW1 pad 1: Net-(U1-VBAT+) -> Net-(J1-Pin_2)
- SW1 pad 2: Net-(J1-Pin_2) -> Net-(SW1-B)
- SW1 pad 3: (no net) -> unconnected-(SW1-C-Pad3)
- U1 pad 24: Net-(U1-VBAT+) -> Net-(SW1-B)
Routing:
- net ROW_0: track 0.00 -> 252.9 mm, vias 0 -> 1
- net ROW_4: track 0.00 -> 250.0 mm
- net COL_A: track 0.00 -> 238.9 mm, vias 0 -> 1
- net ROW_3: track 0.00 -> 232.4 mm
- net ROW_2: track 0.00 -> 226.5 mm
- net ROW_1: track 0.00 -> 220.2 mm, vias 0 -> 1
- net COL_B: track 0.00 -> 193.4 mm, vias 0 -> 1
- net COL_F: track 0.00 -> 192.9 mm, vias 0 -> 2
- net COL_E: track 0.00 -> 184.1 mm, vias 0 -> 2
- net COL_C: track 0.00 -> 174.7 mm, vias 0 -> 1
- net COL_I: track 0.00 -> 155.0 mm, vias 0 -> 1
- net COL_J: track 0.00 -> 150.4 mm, vias 0 -> 1
- net COL_H: track 0.00 -> 148.8 mm, vias 0 -> 1
- net COL_K: track 0.00 -> 148.7 mm, vias 0 -> 1
- net COL_D: track 0.00 -> 135.0 mm, vias 0 -> 1
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Other:
- board size 140.3 x 111.5 mm -> 167.7 x 112.3 mm
- board text added: "AQChron"
- board text added: "LENIMAL PCB DESIGN 01.2025"
- board text added: "Split Staggered Ortholinear Keyboard"

Commit message: updated version, ready for production (v1)
Parts:
- moved J2 1.50 mm to (55.5, 86.0)
- moved SW1 0.15 mm to (84.8, 51.8)
Routing:
- net Net-(U1-NRST): track 18.1 -> 21.7 mm
- net COL_I: track 155.0 -> 152.4 mm
- net VW_CS: track 12.6 -> 14.9 mm
- net COL_A: track 238.9 -> 239.9 mm
- net Net-(SW1-B): track 16.2 -> 17.2 mm
- net GNDREF: vias 19 -> 25
Other:
- board text added: "+"
- board text added: "-"
- board text added: "R0CA"
- board text added: "R0CB"
- board text added: "R0CC"
- board text added: "R0CE"
- board text added: "R0CF"
- board text added: "R0CG"
- board text added: "R1CA"
- board text added: "R1CB"
- board text added: "R1CC"
- board text added: "R1CD"
- board text added: "R1CE"
- board text added: "R1CF"
- board text added: "R1CG"
- board text added: "R2CA"
- board text added: "R2CB"
- board text added: "R2CC"
- board text added: "R2CD"
- board text added: "R2CE"
- board text added: "R2CF"
- board text added: "R2CG"
- board text added: "R3CA"
- board text added: "R3CB"
- board text added: "R3CC"
- board text added: "R3CD"
- board text added: "R3CE"
- board text added: "R3CF"
- board text added: "R3CG"
- board text added: "R4CA"
- board text added: "R4CB"
- board text added: "R4CC"
- board text added: "R4CD"
- board text added: "R4CE"
- board text added: "R4CF"
- board text added: "R4CG"
