File: hardware/keyboard.kicad_pcb (KiCad board)
At the start: 2 copper layers, 145.2 x 112.3 mm, 84 parts, among them J1 BATT, J2 nice!view, SW1 PLAY/PAUSE, SW10 NEXT, SW11 TAB, SW12 Q, SW13 W, SW14 E, SW15 R, SW16 T, SW17 CAPS, SW18 A, SW19 S, SW2 TILDA, SW20 D, SW21 F, SW22 G, SW23 M2, SW24 SHIFT, SW25 Z, SW26 X, SW27 C, SW28 V, SW29 B, SW3 1, SW30 ALT_1, SW31 FN, SW32 CONTROL, SW33 OPTION, SW34 COMMAND, SW35 SPACE, SW4 2, SW5 3, SW6 4, SW7 5, SW8 ON_OFF, SW9 NRST, U1 nice!nano

Commit message: finish right keyboard, generate 3D models, add distribution folders
Parts:
- J1: footprint Connector_JST:JST_ZH_B2B-ZR_1x02_P1.50mm_Vertical -> Connector_JST:JST_PH_S2B-PH-K_1x02_P2.00mm_Horizontal
- SW8: footprint Button_Switch_THT:SW_Slide_SPDT_Angled_CK_OS102011MA1Q -> ScottoKeebs_Components:Switch_MSK12C02
- moved G*** 12.5 mm to (105.8, 140.8) (x2)
- moved J1 3.61 mm to (140.0, 55.0), turned to 90 degrees
- moved SW8 1.27 mm to (146.8, 51.8), turned to 0 degrees
Routing:
- net Net-(J1-Pin_2): track 13.8 -> 10.3 mm
- net Net-(SW8-B): track 36.2 -> 35.1 mm
Other:
- board text added: "AQChron"
- board text added: "LENIMAL PCB DESIGN 01.2025"

Commit message: updated version, ready for production (v1)
Routing:
- net COL_E: track 133.6 -> 134.7 mm
Other:
- board text added: "+"
- board text added: "-"
- board text added: "R0CA"
- board text added: "R0CC"
- board text added: "R0CF"
- board text added: "R0CG"
- board text added: "R1CA"
- board text added: "R1CB"
- board text added: "R1CC"
- board text added: "R1CD"
- board text added: "R1CE"
- board text added: "R1CF"
- board text added: "R1CG"
- board text added: "R2CA"
- board text added: "R2CB"
- board text added: "R2CC"
- board text added: "R2CD"
- board text added: "R2CE"
- board text added: "R2CF"
- board text added: "R2CG"
- board text added: "R3CA"
- board text added: "R3CB"
- board text added: "R3CC"
- board text added: "R3CD"
- board text added: "R3CE"
- board text added: "R3CF"
- board text added: "R3CG"
- board text added: "R4CA"
- board text added: "R4CB"
- board text added: "R4CC"
- board text added: "R4CD"
- board text added: "R4CE"
- board text added: "R4CF"
- board text added: "R4CG"
